File: PHOBOS/PHOBOS_Control/_restore_backup_2026-08-24T00-13-26-124/PHOBOS_Control.kicad_pcb (KiCad board)
At the start: 2 copper layers, 125.4 x 71.6 mm, 76 parts, among them J1 Screw_Terminal_01x02, J2 Conn_01x06, J3 Conn_Coaxial, J5 DE9_Pins_MountingHoles, J6 USB4056-03-A_REVA2, U1 SX1280IMLTRT, U2 TLV9351IDCKR, U3 W25Q128JVSIQ, U4 NCP1117-3.3_SOT223, U5 RP2040, U6 TLV9351IDCKR, U7 TLV9351IDCKR, U8 TLV9351IDCKR, Y1 ABM8-272-T3, Y2 C1E-52.000-10-1012-X-M

Commit message: Layout and routing began
Parts:
- moved J6 46.4 mm to (135.0, 403.7), turned to 0 degrees
- moved R11 43.9 mm to (140.8, 400.2), turned to -90 degrees
- moved J2 40.5 mm to (135.0, 351.7)
- moved J1 32.8 mm to (68.5, 369.7)
- moved R21 29.8 mm to (135.5, 395.1), turned to 90 degrees
- moved R19 29.5 mm to (134.5, 395.1), turned to 90 degrees
- moved R10 28.9 mm to (133.3, 395.1), turned to 90 degrees
- moved C13 22.6 mm to (82.8, 361.6)
- moved C14 22.6 mm to (79.5, 361.6)
- moved C12 22.6 mm to (81.2, 361.6)
- moved U4 22.3 mm to (79.8, 355.2)
- moved R9 20.6 mm to (73.0, 361.2), turned to 0 degrees
- moved D5 18.7 mm to (72.1, 362.6), turned to 0 degrees
- moved D4 10.7 mm to (90.8, 371.8), turned to 0 degrees
- moved D1 10.0 mm to (90.8, 369.2), turned to 0 degrees
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Routing:
- net VIN: track 6.33 -> 0.00 mm
- net +BATT: track 4.14 -> 0.00 mm
- net /USB_D+: track 0.00 -> 2.01 mm
- net /USB_D-: track 0.00 -> 2.01 mm
- net Net-(D5-A): track 1.60 -> 0.00 mm
- removed copper zone on F.Cu, net +3V3
Other:
- board size 125.4 x 71.6 mm -> 1 x 0.6 mm
