File: PHOBOS/Transceiver/Transceiver.kicad_sch (KiCad schematic)
At the start: 18 parts, among them J1 Conn_01x06, J2 Conn_Coaxial, U1 SX1280IMLTRT, Y1 C1E-52.000-10-1012-X-M

Commit message: Initial PCB layout updated.
Connections:
- net NSS: now also J1.1 (Pin_1); no longer J1.5 (Pin_5)
- net VDD: now also C10.1, J1.5 (Pin_5), U1.15 (VBAT); no longer J1.1 (Pin_1)
- net XTA: now reaches U1.4 (XTA), Y1.1
- net XTB: now reaches U1.6 (XTB), Y1.3
- net VR_PA: now reaches C5.1, U1.1 (VR_PA)
- net DCC_FB: now reaches C6.1, C9.1, L4.2, U1.12 (DCC_FB), U1.2 (VDD_IN)
- net RFIO: now reaches C0.1, L1.1, U1.22 (RFIO)
- net VBAT_IO: now reaches C8.1, R15.1, U1.11 (VBAT_IO)
- net DCC_SW: now reaches L4.1, U1.14 (DCC_SW)
- net ANTENNA: now reaches C3.2, J2.1 (In)
Other:
- moved on the sheet: C8

Commit message: design blocks tested. connectors added
Parts:
- J1: now not fitted; now left out of the parts list
- J2: footprint Connector_Coaxial:SMA_Amphenol_132134-10_Vertical -> SMA_J_P_GF_RA_SM1:SAMTEC_SMA-J-P-GF-RA-SM1
Connections:
- net GND: now also J2.3, J2.4, J2.5
- net VDD renamed +3.3V
