File: PHOBOS/Transceiver/sx1280.kicad_block/sx1280.kicad_pcb (KiCad board)
At the start: 2 copper layers, 24.2 x 15.6 mm, 17 parts, among them J2 Conn_Coaxial, U1 SX1280IMLTRT, Y1 C1E-52.000-10-1012-X-M

Commit message: mounting holes added and shape changed. design blocks utilized
Other:
- board outline removed
