File: PHOBOS/PHOBOS_Control/_restore_backup_2026-08-29T01-29-52-489/PHOBOS_Control.kicad_pcb (KiCad board)
At the start: 2 copper layers, 34.7 x 49.9 mm, 76 parts, among them J2 Conn_Coaxial, J3 USB4056-03-A_REVA2, J4 Screw_Terminal_01x02, J7 Conn_01x05, J8 Conn_01x02, U1 SX1280IMLTRT, U2 W25Q128JVSIQ, U3 NCP1117-3.3_SOT223, U4 RP2040, U5 TLV9351IDCKR, U6 TLV9351IDCKR, U7 TLV9351IDCKR, U8 TLV9351IDCKR, Y1 C1E-52.000-10-1012-X-M, Y2 ABM8-272-T3

Commit message: ground plane thermal releif added
Routing:
- net GND: track 26.8 -> 10.5 mm, vias 169 -> 168
Changed lines of the file:
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@@
 	)
 	(segment
-		(start 163.676005 113.9075)
-		(end 163.641005 113.9075)
-		(width 0.2)
-		(layer "F.Cu")
-		(net "GND")
-	)
-	(segment
 		(start 151.739006 108.0755)
 		(end 150.689005 108.075499)
@@
 	)
 	(segment
-		(start 163.518505 101.6465)
-		(end 164.416505 101.6465)
-		(width 0.2)
-		(layer "F.Cu")
-		(net "GND")
-	)
-	(segment
-		(start 163.356506 105.4565)
-		(end 164.416505 105.4565)
-		(width 0.2)
-		(layer "F.Cu")
-		(net "GND")
-	)
-	(segment
-		(start 157.701924 108.867358)
-		(end 157.701924 106.463196)
-		(width 0.381)
-		(layer "F.Cu")
-		(net "GND")
-	)
-	(segment
-		(start 163.950003 113.5845)
-		(end 164.924505 113.5845)
-		(width 0.2)
-		(layer "F.Cu")
-		(net "GND")
-	)
-	(segment
 		(start 146.689003 107.575502)
 		(end 147.439005 107.5755)
@@
 	)
 	(segment
-		(start 151.6545 99.752003)
-		(end 151.792004 99.614499)
-		(width 0.2)
-		(layer "F.Cu")
-		(net "GND")
-	)
-	(segment
 		(start 155.475003 104.6945)
 		(end 156.3445 103.825003)
@@
 	)
 	(segment
-		(start 162.456505 107.2565)
-		(end 162.456505 106.356501)
-		(width 0.2)
-		(layer "F.Cu")
-		(net "GND")
-	)
-	(segment
-		(start 163.634004 113.900499)
-		(end 163.950003 113.5845)
-		(width 0.2)
-		(layer "F.Cu")
-		(net "GND")
-	)
-	(segment
 		(start 156.3445 103.825003)
 		(end 156.3445 102.6915)
@@
 	)
 	(segment
-		(start 162.456505 106.356501)
-		(end 163.003506 105.8095)
-		(width 0.2)
-		(layer "F.Cu")
-		(net "GND")
-	)
-	(segment
-		(start 143.134004 107.488)
-		(end 143.134004 106.400499)
-		(width 0.2)
-		(layer "F.Cu")
-		(net "GND")
-	)
-	(segment
-		(start 163.521998 110.1265)
-		(end 163.873998 109.7745)
-		(width 0.2)
-		(layer "F.Cu")
-		(net "GND")
-	)
-	(segment
-		(start 144.271505 108.625501)
-		(end 143.134004 107.488)
-		(width 0.2)
-		(layer "F.Cu")
-		(net "GND")
-	)
-	(segment
 		(start 147.439005 107.5755)
 		(end 148.689005 108.8255)
@@
 	)
 	(segment
-		(start 151.6545 100.229)
-		(end 151.6545 99.752003)
-		(width 0.2)
-		(layer "F.Cu")
-		(net "GND")
-	)
-	(segment
-		(start 162.456505 107.2565)
-		(end 163.323504 108.123499)
-		(width 0.2)
-		(layer "F.Cu")
-		(net "GND")
-	)
-	(segment
 		(start 152.149005 107.665501)
 		(end 151.739006 108.0755)
@@
 	)
 	(segment
-		(start 163.323504 108.123499)
-		(end 164.492004 108.123499)
-		(width 0.2)
-		(layer "F.Cu")
-		(net "GND")
-	)
-	(segment
 		(start 154.332005 104.6945)
 		(end 155.475003 104.6945)
@@
 	)
 	(segment
-		(start 157.701924 106.463196)
-		(end 157.34837 106.109642)
-		(width 0.381)
-		(layer "F.Cu")
-		(net "GND")
-	)
-	(segment
-		(start 163.641005 113.9075)
-		(end 163.634004 113.900499)
-		(width 0.2)
-		(layer "F.Cu")
-		(net "GND")
-	)
-	(segment
-		(start 163.138505 102.0265)
-		(end 163.518505 101.6465)
-		(width 0.2)
-		(layer "F.Cu")
-		(net "GND")
-	)
-	(segment
-		(start 163.003506 105.8095)
-		(end 163.356506 105.4565)
-		(width 0.2)
-		(layer "F.Cu")
-		(net "GND")
-	)
-	(segment
-		(start 163.873998 109.7745)
-		(end 164.8975 109.7745)
-		(width 0.2)
-		(layer "F.Cu")
-		(net "GND")
-	)
-	(segment
 		(start 165.111504 87.321999)
 		(end 167.057004 85.376499)
@@
 	)
 	(via
-		(at 143.134004 106.400499)
-		(size 0.6)
-		(drill 0.3)
-		(layers "F.Cu" "B.Cu")
-		(free yes)
-		(net "GND")
-	)
-	(via
 		(at 152.239005 124.825501)
 		(size 0.6)
@@
 	)
 	(segment
-		(start 161.702 92.375499)
-		(end 161.702 95.4645)
-		(width 0.2)
-		(layer "F.Cu")
-		(net "+3V3")
-	)
-	(segment
 		(start 158.048 93.341999)
 		(end 157.7445 93.645499)
@@
 	)
 	(segment
-		(start 161.702 95.4645)
-		(end 162.0545 95.817)
-		(width 0.2)
-		(layer "F.Cu")
-		(net "+3V3")
-	)
-	(segment
 		(start 153.682 96.429)
 		(end 153.907 96.654)
@@
 	)
 	(segment
+		(start 161.702 92.375499)
+		(end 161.702 95.4645)
+		(width 0.2)
+		(layer "F.Cu")
+		(net "+3V3")
+	)
+	(segment
 		(start 168.574505 83.687526)
 		(end 168.333007 83.446028)
@@
 	)
 	(segment
+		(start 161.702 95.4645)
+		(end 162.0545 95.817)
+		(width 0.2)
+		(layer "F.Cu")
+		(net "+3V3")
+	)
+	(segment
 		(start 163.857004 87.904)
 		(end 165.000005 89.047001)
@@
 	)
 	(segment
-		(start 169.014004 105.3955)
-		(end 172.305005 105.3955)
+		(start 163.126005 101.054)
+		(end 163.138505 101.0665)
 		(width 0.2)
 		(layer "F.Cu")
-		(net "/PS1")
+		(net "/PS1MCU")
 	)
 	(segment
-		(start 166.091505 103.369)
-		(end 166.014005 103.4465)
+		(start 160.782 101.054)
+		(end 163.126005 101.054)
 		(width 0.2)
 		(layer "F.Cu")
-		(net "/PS1")
+		(net "/PS1MCU")
 	)
 	(segment
-		(start 167.051004 103.4465)
-		(end 167.058004 103.4395)
+		(start 164.346506 101.0665)
+		(end 164.416505 100.996501)
 		(width 0.2)
 		(layer "F.Cu")
-		(net "/PS1")
+		(net "/PS1MCU")
 	)
 	(segment
-		(start 166.091505 102.296499)
-		(end 166.091505 103.369)
+		(start 163.138505 101.0665)
+		(end 164.346506 101.0665)
 		(width 0.2)
 		(layer "F.Cu")
-		(net "/PS1")
+		(net "/PS1MCU")
 	)
 	(segment
-		(start 167.058004 103.4395)
-		(end 169.014004 105.3955)
+		(start 164.416505 102.296499)
+		(end 164.416505 103.044)
 		(width 0.2)
 		(layer "F.Cu")
-		(net "/PS1")
+		(net "Net-(U8--)")
 	)
 	(segment
-		(start 166.014005 103.4465)
-		(end 167.051004 103.4465)
+		(start 163.614005 103.4465)
+		(end 164.819005 103.4465)
 		(width 0.2)
 		(layer "F.Cu")
-		(net "/PS1")
+		(net "Net-(U8--)")
 	)
 	(segment
-		(start 163.126005 101.054)
-		(end 163.138505 101.0665)
+		(start 164.416505 103.044)
+		(end 164.819005 103.4465)
 		(width 0.2)
 		(layer "F.Cu")
-		(net "/PS1MCU")
+		(net "Net-(U8--)")
 	)
 	(segment
-		(start 160.782 101.054)
-		(end 163.126005 101.054)
+		(start 169.014004 105.3955)
+		(end 172.305005 105.3955)
 		(width 0.2)
 		(layer "F.Cu")
-		(net "/PS1MCU")
+		(net "/PS1")
 	)
 	(segment
-		(start 164.346506 101.0665)
-		(end 164.416505 100.996501)
+		(start 166.091505 103.369)
+		(end 166.014005 103.4465)
 		(width 0.2)
 		(layer "F.Cu")
-		(net "/PS1MCU")
+		(net "/PS1")
 	)
 	(segment
-		(start 163.138505 101.0665)
-		(end 164.346506 101.0665)
+		(start 167.051004 103.4465)
+		(end 167.058004 103.4395)
 		(width 0.2)
 		(layer "F.Cu")
-		(net "/PS1MCU")
+		(net "/PS1")
 	)
 	(segment
-		(start 164.416505 102.296499)
-		(end 164.416505 103.044)
+		(start 166.091505 102.296499)
+		(end 166.091505 103.369)
 		(width 0.2)
 		(layer "F.Cu")
-		(net "Net-(U8--)")
+		(net "/PS1")
 	)
 	(segment
-		(start 163.614005 103.4465)
-		(end 164.819005 103.4465)
+		(start 167.058004 103.4395)
+		(end 169.014004 105.3955)
 		(width 0.2)
 		(layer "F.Cu")
-		(net "Net-(U8--)")
+		(net "/PS1")
 	)
 	(segment
-		(start 164.416505 103.044)
-		(end 164.819005 103.4465)
+		(start 166.014005 103.4465)
+		(end 167.051004 103.4465)
 		(width 0.2)
 		(layer "F.Cu")
-		(net "Net-(U8--)")
+		(net "/PS1")
 	)
 	(segment
@@
 		(hatch edge 0.5)
 		(priority 1)
-		(connect_pads
+		(connect_pads yes
 			(clearance 0.127)
 		)
@@
 			"138c03bf-1c43-4082-961f-7e6c2393e215" "187049e9-e7e5-4c11-b618-d12b84ddf737"
 			"21e4ec1b-309d-494a-9234-8223c6da6371" "28833abe-e432-4abf-9a99-5948f0719dac"
-			"2b785a23-cdd9-4113-8c73-e28a99385dc5" "37c9876f-b9d8-463a-bb57-c0785a9e78a4"
-			"39846bc8-e13a-4645-8bcd-1957753c30ea" "3c77c619-b7cd-47b7-9500-ccb6c6b41163"
-			"45eb3213-5030-43ae-9643-49a4a956731a" "48741bf4-95f3-4b8f-890d-5827e1270a86"
+			"37c9876f-b9d8-463a-bb57-c0785a9e78a4" "39846bc8-e13a-4645-8bcd-1957753c30ea"
+			"3c77c619-b7cd-47b7-9500-ccb6c6b41163" "45eb3213-5030-43ae-9643-49a4a956731a"
 			"4b55cf10-3af5-4dbe-8a3b-79008d56f5e2" "4e6019b1-3f37-40c0-a5ff-8048f310d9f3"
 			"523bdea2-00d8-440b-bfbd-bd4f83ce3bd6" "59e81c85-9419-4de1-982b-2580cec341e9"
@@
 			"663c0740-1076-4911-88eb-ff280ea90020" "6b16d792-056c-4567-8b5c-3a12483df3a1"
 			"6c95634d-62aa-4c81-9b5f-0c4b3cfe3719" "6d63aa82-71d0-482b-817d-126f8f5e5e70"
-			"72447b0e-a1c5-4c68-a00a-44be1682d4db" "733a0b12-0017-4c6d-9c68-afa1b4d184b4"
-			"82475803-6d4f-4c20-bb33-185f2e3e5d78" "9477905c-f0a2-4971-abb4-aad747cd85f7"
-			"a2807391-10ea-4b8f-9808-e0642ca56e64" "a2df16ac-9b50-4902-b0e5-299d8c1dd6e2"
-			"a3445366-e813-421a-8c92-6792b400d440" "a47f245b-31a7-41a1-ac40-bca3187ded5d"
-			"af5d6e31-e499-41e6-a22e-9cfe0004e232" "b30a7736-1e93-4425-9c89-c34faaf46e41"
-			"ba04cea6-54cf-4025-bcbf-b7bdc638c5a0" "c3203430-e423-45bb-8d67-094fa16793d8"
-			"c834ae8e-9ef8-45a0-b1c3-8e49ece051e2" "cc00126d-0169-4edc-907a-918cde04bd20"
-			"ce840980-d04a-409a-9e06-d926ad90c864" "e0f74305-aa27-4136-80f8-40a694adc117"
+			"6d6e4268-d2b9-40ce-954c-cb1ce679d01a" "72447b0e-a1c5-4c68-a00a-44be1682d4db"
+			"733a0b12-0017-4c6d-9c68-afa1b4d184b4" "82475803-6d4f-4c20-bb33-185f2e3e5d78"
+			"9477905c-f0a2-4971-abb4-aad747cd85f7" "a2807391-10ea-4b8f-9808-e0642ca56e64"
+			"a2df16ac-9b50-4902-b0e5-299d8c1dd6e2" "a3445366-e813-421a-8c92-6792b400d440"
+			"a47f245b-31a7-41a1-ac40-bca3187ded5d" "af5d6e31-e499-41e6-a22e-9cfe0004e232"
+			"b30a7736-1e93-4425-9c89-c34faaf46e41" "ba04cea6-54cf-4025-bcbf-b7bdc638c5a0"
+			"c3203430-e423-45bb-8d67-094fa16793d8" "c834ae8e-9ef8-45a0-b1c3-8e49ece051e2"
+			"cc00126d-0169-4edc-907a-918cde04bd20" "ce840980-d04a-409a-9e06-d926ad90c864"
+			"db30af35-3cfd-474b-a33b-579dd35c0054" "e0f74305-aa27-4136-80f8-40a694adc117"
 			"e8bb712d-b58f-483f-b7c2-7e8d080b73cc" "f6b34500-503b-48b1-a538-cbc65e7d2617"
 			"fa4d31b9-281e-4bcf-89d9-5d7129d302a5" "fc64ee87-0fe8-441c-bafc-275009d19d5f"
