File: PHOBOS/PHOBOS_RF_Digital/PHOBOS_RF_Digital.kicad_pcb (KiCad board)
At the start: 4 copper layers, 303 x 142.8 mm, 28 parts, among them IC1 PD2328J5050S2HF, IC2 PD2328J5050S2HF, IC3 PD2328J5050S2HF, IC4 MAPS-010144-TR0500, IC5 MAPS-010144-TR0500, IC6 MAPS-010144-TR0500, IC7 MAPS-010144-TR0500, J1 RF_IN, J2 PS1, J4 PS2, J5 PS3, J6 PS4, J7 PWR

Commit message: Refactored for later organization and bibliographies fixed (now references.bib)
Parts:
- removed AE1 (x2), AE2 (x2), AE3 (x2), AE4 (x2): Antenna, 2.4GHz_Patch_Antenna:Patch_Antenna
- moved IC6 50.2 mm to (74.0, 52.0)
- moved J4 50.2 mm to (87.9, 38.3)
- moved J6 50.2 mm to (96.0, 38.3)
- moved TP1 50.2 mm to (79.5, 38.6)
- moved TP3 50.2 mm to (79.5, 47.9)
- moved IC5 50.2 mm to (74.0, 45.7)
- moved J5 50.2 mm to (91.9, 38.3)
- moved TP4 50.2 mm to (79.5, 52.6)
- moved IC7 50.2 mm to (74.0, 58.3)
- moved TP2 50.2 mm to (79.5, 43.3)
- moved J2 50.2 mm to (83.8, 38.3)
- moved J7 42.8 mm to (109.5, 43.4)
- moved IC3 9.31 mm to (134.6, 100.0)
- moved J1 9.31 mm to (121.5, 102.0)
- moved R2 9.31 mm to (141.0, 129.7)
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Other:
- board size 303 x 142.8 mm -> 167 x 107.5 mm
- board text removed: "Not Properly Layed Out"

Commit message: RF board continued for general size estimates
Parts:
- added AE1: Antenna, 2.4GHz_Patch_Antenna:Patch_Antenna, F.Cu at (183.3, 123.5)
- added AE1: Antenna, 2.4GHz_Patch_Antenna:Patch_Antenna, F.Cu at (315.7, 123.5)
- added AE2: Antenna, 2.4GHz_Patch_Antenna:Patch_Antenna, F.Cu at (381.9, 123.5)
- added AE2: Antenna, 2.4GHz_Patch_Antenna:Patch_Antenna, F.Cu at (249.5, 123.5)
- added AE3: Antenna, 2.4GHz_Patch_Antenna:Patch_Antenna, F.Cu at (249.5, 48.2)
- added AE3: Antenna, 2.4GHz_Patch_Antenna:Patch_Antenna, F.Cu at (381.9, 48.2)
- added AE4: Antenna, 2.4GHz_Patch_Antenna:Patch_Antenna, F.Cu at (315.7, 48.2)
- added AE4: Antenna, 2.4GHz_Patch_Antenna:Patch_Antenna, F.Cu at (183.3, 48.2)
- moved IC6 50.2 mm to (123.6, 59.7)
- moved J4 50.2 mm to (137.5, 46.0)
- moved J6 50.2 mm to (145.6, 46.0)
- moved TP1 50.2 mm to (129.1, 46.3)
- moved TP3 50.2 mm to (129.1, 55.6)
- moved IC5 50.2 mm to (123.6, 53.4)
- moved J5 50.2 mm to (141.5, 46.0)
- moved TP4 50.2 mm to (129.1, 60.2)
- moved IC7 50.2 mm to (123.6, 66.0)
- moved TP2 50.2 mm to (129.1, 50.9)
- moved J2 50.2 mm to (133.4, 46.0)
- moved J7 42.8 mm to (152.1, 47.7)
- moved IC3 9.31 mm to (136.9, 91.0)
- moved J1 9.31 mm to (123.8, 93.0)
- moved R2 9.31 mm to (143.3, 120.7)
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Other:
- board size 167 x 107.5 mm -> 303 x 142.8 mm
- board text added: "Not Properly Layed Out"
