File: PHOBOS/PHOBOS_RF_Digital/PHOBOS_RF_Digital.kicad_sch (KiCad schematic)
At the start: 24 parts, among them IC1 PD2328J5050S2HF, IC2 PD2328J5050S2HF, IC3 PD2328J5050S2HF, IC4 MAPS-010144-TR0500, IC5 MAPS-010144-TR0500, IC6 MAPS-010144-TR0500, IC7 MAPS-010144-TR0500, J1 RF_IN, J2 PS1, J4 PS2, J5 PS3, J6 PS4, J7 PWR

Commit message: RF board continued for general size estimates
Parts:
- AE1, AE2, AE3, AE4: footprint (none) -> 2.4GHz_Patch_Antenna:Patch_Antenna
- IC4, IC5, IC6, IC7: footprint QFN50P400X400X100-25N-D -> MAPS-010144-TR0500:QFN50P400X400X100-25N-D
Changed lines of the file:
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@@
 			)
 		)
-		(property "Footprint" ""
+		(property "Footprint" "2.4GHz_Patch_Antenna:Patch_Antenna"
 			(at 424.18 81.28 0)
 			(hide yes)
@@
 			)
 		)
-		(property "Footprint" ""
+		(property "Footprint" "2.4GHz_Patch_Antenna:Patch_Antenna"
 			(at 426.72 316.23 0)
 			(hide yes)
@@
 			)
 		)
-		(property "Footprint" "QFN50P400X400X100-25N-D"
+		(property "Footprint" "MAPS-010144-TR0500:QFN50P400X400X100-25N-D"
 			(at 400.05 320.98 0)
 			(hide yes)
@@
 			)
 		)
-		(property "Footprint" ""
+		(property "Footprint" "2.4GHz_Patch_Antenna:Patch_Antenna"
 			(at 425.45 168.91 0)
 			(hide yes)
@@
 			)
 		)
-		(property "Footprint" ""
+		(property "Footprint" "2.4GHz_Patch_Antenna:Patch_Antenna"
 			(at 426.72 242.57 0)
 			(hide yes)
@@
 			)
 		)
-		(property "Footprint" "QFN50P400X400X100-25N-D"
+		(property "Footprint" "MAPS-010144-TR0500:QFN50P400X400X100-25N-D"
 			(at 400.05 394.64 0)
 			(hide yes)
@@
 			)
 		)
-		(property "Footprint" "QFN50P400X400X100-25N-D"
+		(property "Footprint" "MAPS-010144-TR0500:QFN50P400X400X100-25N-D"
 			(at 398.78 247.32 0)
 			(hide yes)
@@
 			)
 		)
-		(property "Footprint" "QFN50P400X400X100-25N-D"
+		(property "Footprint" "MAPS-010144-TR0500:QFN50P400X400X100-25N-D"
 			(at 397.51 159.69 0)
 			(hide yes)

Commit message: Refactored for later organization and bibliographies fixed (now references.bib)
Parts:
- AE1, AE2, AE3, AE4: footprint 2.4GHz_Patch_Antenna:Patch_Antenna -> (none)
- IC4, IC5, IC6, IC7: footprint MAPS-010144-TR0500:QFN50P400X400X100-25N-D -> QFN50P400X400X100-25N-D
Changed lines of the file:
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@@
 			)
 		)
-		(property "Footprint" "2.4GHz_Patch_Antenna:Patch_Antenna"
+		(property "Footprint" ""
 			(at 424.18 81.28 0)
 			(hide yes)
@@
 			)
 		)
-		(property "Footprint" "2.4GHz_Patch_Antenna:Patch_Antenna"
+		(property "Footprint" ""
 			(at 426.72 316.23 0)
 			(hide yes)
@@
 			)
 		)
-		(property "Footprint" "MAPS-010144-TR0500:QFN50P400X400X100-25N-D"
+		(property "Footprint" "QFN50P400X400X100-25N-D"
 			(at 400.05 320.98 0)
 			(hide yes)
@@
 			)
 		)
-		(property "Footprint" "2.4GHz_Patch_Antenna:Patch_Antenna"
+		(property "Footprint" ""
 			(at 425.45 168.91 0)
 			(hide yes)
@@
 			)
 		)
-		(property "Footprint" "2.4GHz_Patch_Antenna:Patch_Antenna"
+		(property "Footprint" ""
 			(at 426.72 242.57 0)
 			(hide yes)
@@
 			)
 		)
-		(property "Footprint" "MAPS-010144-TR0500:QFN50P400X400X100-25N-D"
+		(property "Footprint" "QFN50P400X400X100-25N-D"
 			(at 400.05 394.64 0)
 			(hide yes)
@@
 			)
 		)
-		(property "Footprint" "MAPS-010144-TR0500:QFN50P400X400X100-25N-D"
+		(property "Footprint" "QFN50P400X400X100-25N-D"
 			(at 398.78 247.32 0)
 			(hide yes)
@@
 			)
 		)
-		(property "Footprint" "MAPS-010144-TR0500:QFN50P400X400X100-25N-D"
+		(property "Footprint" "QFN50P400X400X100-25N-D"
 			(at 397.51 159.69 0)
 			(hide yes)
