File: PHOBOS/PHOBOS_RF_Digital/PHOBOS_RF_Digital.kicad_sch (KiCad schematic)
At the start: 24 parts, among them IC1 PD2328J5050S2HF, IC2 PD2328J5050S2HF, IC3 PD2328J5050S2HF, IC4 MAPS-010144-TR0500, IC5 MAPS-010144-TR0500, IC6 MAPS-010144-TR0500, IC7 MAPS-010144-TR0500, J1 RF_IN, J2 PS1, J4 PS2, J5 PS3, J6 PS4, J7 PWR

Commit message: mounting holes added. 1x4 design began
Parts:
- added H1, H2, H3, H4: MountingHole, MountingHole:MountingHole_3.2mm_M3, symbol Mechanical:MountingHole
