File: PHOBOS/PHOBOS_RF_Digital/PHOBOS_RF_Digital.kicad_sch (KiCad schematic)
At the start: 28 parts, among them IC1 PD2328J5050S2HF, IC2 PD2328J5050S2HF, IC3 PD2328J5050S2HF, IC4 MAPS-010144-TR0500, IC5 MAPS-010144-TR0500, IC6 MAPS-010144-TR0500, IC7 MAPS-010144-TR0500, J1 RF_IN, J2 PS1, J4 PS2, J5 PS3, J6 PS4, J7 PWR

Commit message: 4 SMA version started.
Parts:
- removed J2: PS1, Connector_PinSocket_2.00mm:PinSocket_1x05_P2.00mm_Vertical, symbol Connector_Generic:Conn_01x05
- removed J4: PS2, Connector_PinSocket_2.00mm:PinSocket_1x05_P2.00mm_Vertical, symbol Connector_Generic:Conn_01x05
- removed J5: PS3, Connector_PinSocket_2.00mm:PinSocket_1x05_P2.00mm_Vertical, symbol Connector_Generic:Conn_01x05
- removed J6: PS4, Connector_PinSocket_2.00mm:PinSocket_1x05_P2.00mm_Vertical, symbol Connector_Generic:Conn_01x05
- added J3: PS2, Connector_PinHeader_1.00mm:PinHeader_2x04_P1.00mm_Vertical, symbol Connector_Generic:Conn_02x04_Odd_Even
- added J4: PS1, Connector_PinHeader_1.00mm:PinHeader_2x04_P1.00mm_Vertical, symbol Connector_Generic:Conn_02x04_Odd_Even
- added J5: PS3, Connector_PinHeader_1.00mm:PinHeader_2x04_P1.00mm_Vertical, symbol Connector_Generic:Conn_02x04_Odd_Even
- added J6: PS4, Connector_PinHeader_1.00mm:PinHeader_2x04_P1.00mm_Vertical, symbol Connector_Generic:Conn_02x04_Odd_Even
- IC4, IC5, IC6, IC7: footprint QFN50P400X400X100-25N-D -> MAPS-010144-TR0500:QFN50P400X400X100-25N-D
- J7: now not fitted; now left out of the parts list
Connections:
- net +3V3: now also J3.1 (Pin_1), J4.1 (Pin_1), J5.1 (Pin_1), J6.1 (Pin_1)
- net -3V3: now also J3.5 (Pin_5), J4.5 (Pin_5), J5.5 (Pin_5), J6.5 (Pin_5)
- net GND: now also J3.7 (Pin_7), J3.8 (Pin_8), J4.7 (Pin_7), J4.8 (Pin_8), J5.7 (Pin_7), J5.8 (Pin_8), J6.7 (Pin_7), J6.8 (Pin_8)
- net LE1: now also J4.2 (Pin_2)
- net LE2: now also J3.2 (Pin_2)
- net LE3: now also J5.2 (Pin_2)
- net LE4: now also J6.2 (Pin_2)
- net MOSI_1: now also J4.6 (Pin_6)
- net MOSI_2: now also J3.6 (Pin_6)
- net MOSI_3: now also J5.6 (Pin_6)
- net MOSI_4: now also J6.6 (Pin_6)
- net SCK_1: now also J4.4 (Pin_4)
- net SCK_2: now also J3.4 (Pin_4)
- net SCK_3: now also J5.4 (Pin_4)
- net SCK_4: now also J6.4 (Pin_4)
