File: DEIMOS/INSIGHT/INSIGHT.kicad_sch (KiCad schematic)
At the start: 84 parts, among them J1 Batt, J2 UFL, J3 USB_C_Receptacle_USB2.0_16P, J4 Boot, J5 GND, J6 Stack 1x04, J7 Conn_02x05_Odd_Even, J8 5V, SW3 SW_SPDT, U1 LSM6DS3, U10 453-00139R, U11 MPM3610GQV-Z, U2 MPL3115A2, U3 W25Q128JVSIQ, U5 RP2040, U6 Adafruit GPS, U7 MPM3610GQV-Z, U8 IIS2MDCTR, U9 LoRa Module, Y1 ABM8-272-T3

Commit message: Updated Insight symbols to match formatting of other componets also added notes to add right angle sma port and add bno08x sensor
Connections:
- net GND: no longer U10.11 (GND), U10.2 (GND), U10.21 (GND), U10.24 (GND), U10.25 (GND), U10.26 (GND), U10.28 (GND), U10.29 (GND), U10.30 (GND), U10.31 (GND), U10.35 (GND), U10.4 (GND), U10.40 (GND), U10.41 (GND), U10.42 (GND), U10.43 (GND), U10.44 (GND), U10.45 (GND), U10.46 (GND), U10.47 (GND), U10.7 (GND), U10.9 (GND)
- new net: U10.11 (GND), U10.2 (GND), U10.21 (GND), U10.24 (GND), U10.25 (GND), U10.26 (GND), U10.28 (GND), U10.29 (GND), U10.30 (GND), U10.31 (GND), U10.35 (GND), U10.4 (GND), U10.40 (GND), U10.41 (GND), U10.42 (GND), U10.43 (GND), U10.44 (GND), U10.45 (GND), U10.46 (GND), U10.47 (GND), U10.7 (GND), U10.9 (GND)
Other:
- note added: "Buck Converter"
- note added: "LoRa"
- note added: "This need a right angle sma port routed to it"
- note added: "This needs to be removed and replaced with Bno08x sensor baord"
- moved on the sheet: C26, C27, C28, C3, C4, C5, D10, J2, J6, LS1, R24, R25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

Commit message: General schemtic clean up
Other:
- note added: "This LoRa module is not the one I want to use, I want to use the RM95W"
- moved on the sheet: C1, C10, C11, C12, C13, C14, C15, C16, C17, C18, C19, C2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
