File: DEIMOS/INSIGHT/INSIGHT.kicad_pcb (KiCad board)
At the start: 4 copper layers, 76.8 x 38.1 mm, 76 parts, among them J1 Batt, J2 SMA-J-P-GF-RA-SM1, J3 USB_C_Receptacle_USB2.0_16P, J4 Boot, J5 GND, SW3 SW_SPDT, U1 LSM6DS3, U2 MPL3115A2, U3 W25Q128JVSIQ, U4 BNO085, U5 RP2040, U6 Adafruit GPS, U7 MPM3610GQV-Z, U8 RFM95W-915S2, Y1 ABM8-272-T3, Y2 ABS07-32.768KHZ-1-T

Commit message: Final Final Revisions for now its sleepy time
Connections:
- J2 pad 1: Net-(U8-ANT) -> unconnected-(J2-Pad1)
- U8 pad 9: Net-(U8-ANT) -> unconnected-(U8-ANT-Pad9)
Other:
- board text added: "AURORA Insight V6"
- board text removed: "AURORA Insight"
Changed lines of the file:
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@@
 			(at 0 -3.75 0)
 			(layer "F.SilkS")
+			(hide yes)
 			(effects
 				(font
@@
 		(tags "resistor")
 		(property "Reference" "R35"
-			(at -0.199999 1.2 90)
+			(at -0.63013 1.2 90)
 			(layer "F.SilkS")
 			(effects
@@
 			)
 		)
-		(attr smd)
+		(attr smd dnp)
 		(duplicate_pad_numbers_are_jumpers no)
 		(fp_line
@@
 			(size 1.7 1.7)
 			(layers "F.Cu" "F.Mask" "F.Paste")
-			(net "Net-(U8-ANT)")
+			(net "unconnected-(J2-Pad1)")
 			(pintype "passive")
 			(solder_mask_margin 0.102)
@@
 			(at 0 -3.75 0)
 			(layer "F.SilkS")
+			(hide yes)
 			(effects
 				(font
@@
 			(layers "F.Cu" "F.Mask" "F.Paste")
 			(roundrect_rratio 0.25)
-			(net "Net-(U8-ANT)")
+			(net "unconnected-(U8-ANT-Pad9)")
 			(pinfunction "ANT_9")
 			(pintype "bidirectional")
@@
 			(at 0 -3.75 0)
 			(layer "F.SilkS")
+			(hide yes)
 			(effects
 				(font
@@
 	(footprint "MountingHole:MountingHole_3.2mm_M3_DIN965_Pad"
 		(layer "F.Cu")
-		(at 73.012 51.9035)
+		(at 73.047 51.8935)
 		(descr "Mounting Hole 3.2mm, M3, generated by kicad-footprint-generator mountinghole.py")
 		(tags "mountinghole M3 DIN965")
@@
 			(at 0 -3.75 0)
 			(layer "F.SilkS")
+			(hide yes)
 			(effects
 				(font
@@
 	)
 	(gr_rect
-		(start 67.262 48.1435)
-		(end 144.297 86.211)
+		(start 67.297 48.1435)
+		(end 144.047 86.211)
 		(stroke
 			(width 0.381)
@@
 		(layer "F.SilkS")
 	)
+	(gr_circle
+		(center 72.797 82.3935)
+		(end 75.297 80.3935)
+		(stroke
+			(width 0.1)
+			(type default)
+		)
+		(fill no)
+		(layer "F.SilkS")
+	)
+	(gr_circle
+		(center 73.047 51.8935)
+		(end 75.047 49.3935)
+		(stroke
+			(width 0.1)
+			(type default)
+		)
+		(fill no)
+		(layer "F.SilkS")
+	)
+	(gr_circle
+		(center 139.047 51.8935)
+		(end 141.297 49.6435)
+		(stroke
+			(width 0.1)
+			(type default)
+		)
+		(fill no)
+		(layer "F.SilkS")
+	)
+	(gr_circle
+		(center 139.047 82.3935)
+		(end 141.297 80.1435)
+		(stroke
+			(width 0.1)
+			(type default)
+		)
+		(fill no)
+		(layer "F.SilkS")
+	)
 	(gr_rect
 		(start 67.262 48.0935)
@@
 		)
 	)
-	(gr_text "Nicholas Krupa \n& \nKyle Eckert"
-		(at 85.797 74.1435 0)
+	(gr_text "Mode"
+		(at 71.453 80.927 0)
 		(layer "F.SilkS")
 		(effects
 			(font
 				(size 0.635 0.635)
-				(thickness 0.127)
-				(bold yes)
+				(thickness 0.1524)
 			)
+			(justify left bottom)
 		)
 	)
-	(gr_text "Mode"
-		(at 71.453 80.927 0)
+	(gr_text "AURORA \nInsight V6\n"
+		(at 135.797 75.3935 0)
 		(layer "F.SilkS")
 		(effects
 			(font
-				(size 0.635 0.635)
-				(thickness 0.1524)
+				(size 0.7 0.7)
+				(thickness 0.175)
+				(bold yes)
 			)
-			(justify left bottom)
+			(justify left)
 		)
 	)
-	(gr_text "AURORA Insight\n"
-		(at 103.797 84.6435 0)
+	(gr_text "Nicholas Krupa \n& \nKyle Eckert"
+		(at 138.047 59.1435 0)
 		(layer "F.SilkS")
 		(effects
 			(font
-				(size 0.635 0.635)
-				(thickness 0.15875)
+				(size 0.7 0.7)
+				(thickness 0.175)
 				(bold yes)
 			)
-			(justify left bottom)
 		)
 	)
