File: PHOBOS/COMET/COMET.kicad_pcb (KiCad board)
At the start: 4 copper layers, 63.5 x 25.4 mm, 73 parts, among them J2 M/D, J5 Power/Arm, J6 USB4056-03-A_REVA2, Q1 SISS67DN-T1-GE3, Q2 BSD840N, Q3 SISS67DN-T1-GE3, SW3 KMR211GLFS, U1 MPL3115A2, U2 LSM6DS3, U3 W25Q128JVSIQ, U4 NCP1117-3.3_SOT223, U5 RP2040, Y1 ABM8-272-T3

Commit message: boot pins moved to front, Screw terminals alligned
Parts:
- TP1, TP2: moved to F.Cu
- moved J2 0.13 mm to (113.6, 81.7)
- turned TP1 to 0 degrees
- turned TP2 to 0 degrees
Routing:
- net /QSPI_SS: track 12.2 -> 13.5 mm, vias 1 -> 0

Commit message: Speaker replaced. GND TP fixed.
Parts:
- LS1: footprint Buzzer_Beeper:MagneticBuzzer_PUI_AT-0927-TT-6-R -> OWMB-404020SA-40-17:OWMB-404020SA-40-17
- moved LS1 3.85 mm to (80.5, 62.6)
Routing:
- net GND: track 63.3 -> 65.2 mm, vias 40 -> 41
- net /Speaker: vias 1 -> 2
Other:
- board text added: "GND"
Changed lines of the file:
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@@
 		)
 	)
-	(footprint "Buzzer_Beeper:MagneticBuzzer_PUI_AT-0927-TT-6-R"
+	(footprint "OWMB-404020SA-40-17:OWMB-404020SA-40-17"
 		(layer "F.Cu")
-		(at 82.47 65.891 180)
-		(descr "Buzzer Magnetic 9mm AT-0927-TT-6-R, http://www.puiaudio.com/pdf/AT-0927-TT-6-R.pdf")
-		(tags "Buzzer Magnetic 9mm AT-0927-TT-6-R")
+		(at 80.47 62.596 180)
 		(property "Reference" "LS1"
-			(at 7.708 0.63 270)
+			(at -3 -4.978 180)
+			(unlocked yes)
 			(layer "F.SilkS")
 			(effects
 				(font
-					(size 1 1)
-					(thickness 0.15)
+					(size 0.635 0.635)
+					(thickness 0.1524)
+					(bold yes)
 				)
 			)
 		)
 		(property "Value" "Speaker"
-			(at 2 7 180)
+			(at 0 1 180)
+			(unlocked yes)
 			(layer "F.Fab")
 			(effects
@@
 			(effects
 				(font
-					(size 1.27 1.27)
+					(size 1 1)
 					(thickness 0.15)
 				)
@@
 			(effects
 				(font
-					(size 1.27 1.27)
+					(size 1 1)
 					(thickness 0.15)
 				)
@@
 			)
 		)
-		(attr through_hole)
+		(attr smd)
 		(duplicate_pad_numbers_are_jumpers no)
-		(fp_circle
-			(center 2 0)
-			(end 6.62 0)
+		(fp_line
+			(start -2 -4.35)
+			(end -1.048 -5.366)
 			(stroke
-				(width 0.12)
-				(type solid)
+				(width 0.1)
+				(type default)
 			)
-			(fill no)
 			(layer "F.SilkS")
 		)
-		(fp_circle
-			(center 2 0)
-			(end 6.75 0)
-			(stroke
-				(width 0.05)
-				(type solid)
-			)
-			(fill no)
-			(layer "F.CrtYd")
-		)
-		(fp_circle
-			(center 2 0)
-			(end 6.5 0)
+		(fp_rect
+			(start -2 -5.366)
+			(end 2 -1.366)
 			(stroke
 				(width 0.1)
@@
 			)
 			(fill no)
-			(layer "F.Fab")
-		)
-		(fp_text user "+"
-			(at -1.792 -0.62 180)
 			(layer "F.SilkS")
-			(effects
-				(font
-					(size 1 1)
-					(thickness 0.15)
-				)
-			)
 		)
 		(fp_text user "${REFERENCE}"
-			(at 2 2 180)
-			(layer "F.Fab")
-			(effects
-				(font
-					(size 1 1)
-					(thickness 0.15)
-				)
-			)
-		)
-		(fp_text user "+"
-			(at -1.5 -0.1 180)
+			(at 0 2.5 180)
+			(unlocked yes)
 			(layer "F.Fab")
 			(effects
@@
 			)
 		)
-		(pad "1" thru_hole rect
-			(at 0 0 180)
-			(size 1.6 1.6)
-			(drill 0.9)
-			(layers "*.Cu" "*.Mask")
-			(remove_unused_layers no)
+		(pad "1" smd rect
+			(at -2 -3.366 270)
+			(size 2.4 2)
+			(layers "F.Cu" "F.Mask" "F.Paste")
 			(net "/Speaker")
 			(pinfunction "1_1")
 			(pintype "input")
 		)
-		(pad "2" thru_hole circle
-			(at 4 0 180)
-			(size 1.6 1.6)
-			(drill 0.9)
-			(layers "*.Cu" "*.Mask")
-			(remove_unused_layers no)
+		(pad "2" smd rect
+			(at 2 -3.366 270)
+			(size 2.4 2)
+			(layers "F.Cu" "F.Mask" "F.Paste")
 			(net "GND")
 			(pinfunction "2_2")
@@
 		)
 		(embedded_fonts no)
-		(model "${KICAD10_3DMODEL_DIR}/Buzzer_Beeper.3dshapes/MagneticBuzzer_PUI_AT-0927-TT-6-R.step"
+		(model "${KIPRJMOD}/Parts/OWMB-404020SA-40-17/OWMB-404020SA-40-17_solid_3D.stp"
 			(offset
-				(xyz 0 0 0)
+				(xyz 2.5 3.3 -2.5)
 			)
 			(scale
@@
 			)
 		)
-		(model "${KIPRJMOD}/Parts/AT-0927-TT-6-R/LS_AT-0927-TT-6-R_PUI.step"
-			(hide yes)
-			(offset
-				(xyz 0 0 0)
-			)
-			(scale
-				(xyz 1 1 1)
-			)
-			(rotate
-				(xyz 0 0 0)
-			)
-		)
-		(model "${KIPRJMOD}/Parts/AT-0927-TT-6-R/AT-0927-TT-6-R--3DModel-STEP-461651.STEP"
+		(model "${KICAD9_3DMODEL_DIR}/External_Custom_Parts.3dshapes/OWMB-404020SA-40-17_solid_3D.stp"
 			(offset
-				(xyz 1.9177 0 2.54)
+				(xyz 1.8 3.5 -2.5)
 			)
 			(scale
@@
 			)
 			(rotate
-				(xyz -90 -0 90)
+				(xyz -0 -0 -0)
 			)
 		)
@@
 		)
 	)
+	(gr_text "Boot"
+		(at 92.662 85.245 -0)
+		(layer "F.SilkS")
+		(effects
+			(font
+				(size 0.635 0.635)
+				(thickness 0.1524)
+			)
+		)
+	)
+	(gr_text "GND"
+		(at 99.774 85.245 0)
+		(layer "F.SilkS")
+		(effects
+			(font
+				(size 0.635 0.635)
+				(thickness 0.1524)
+			)
+		)
+	)
 	(gr_text "If You're \nReading This, \nYou've Voided \nYour Warranty..."
 		(at 69.762 73.761 270)
@@
 		)
 	)
-	(gr_text "Boot"
-		(at 92.662 85.245 0)
-		(layer "B.SilkS")
-		(effects
-			(font
-				(size 0.635 0.635)
-				(thickness 0.1524)
-			)
-			(justify mirror)
-		)
-	)
 	(gr_text "DROGUE"
 		(at 115.6236 84.4322 0)
@@
 	)
 	(segment
+		(start 78.47 65.962)
+		(end 78.47 64.449)
+		(width 0.2)
+		(layer "F.Cu")
+		(net "GND")
+	)
+	(segment
 		(start 85.834847 62.261)
 		(end 86.272346 62.698499)
@@
 	)
 	(segment
+		(start 96.98 84.991)
+		(end 97.992 84.991)
+		(width 0.2)
+		(layer "F.Cu")
+		(net "GND")
+	)
+	(segment
 		(start 100.262 67.7833)
 		(end 100.262 67.832178)
@@
 	)
 	(segment
+		(start 78.47 64.449)
+		(end 78.184 64.163)
+		(width 0.2)
+		(layer "F.Cu")
+		(net "GND")
+	)
+	(segment
 		(start 78.012 77.7898)
 		(end 78.1984 77.6034)
@@
 	)
 	(segment
+		(start 97.992 84.991)
+		(end 98.262 85.261)
+		(width 0.2)
+		(layer "F.Cu")
+		(net "GND")
+	)
+	(segment
 		(start 107.1745 77.811)
 		(end 107.1745 77.311001)
@@
 	)
 	(via
+		(at 78.184 64.163)
+		(size 0.5842)
+		(drill 0.2032)
+		(layers "F.Cu" "B.Cu")
+		(net "GND")
+	)
+	(via
 		(at 104.512 67.011)
 		(size 0.5842)
@@
 	)
 	(segment
-		(start 96.98 84.991)
-		(end 97.992 84.991)
-		(width 0.2)
-		(layer "B.Cu")
-		(net "GND")
-	)
-	(segment
-		(start 97.992 84.991)
-		(end 98.262 85.261)
-		(width 0.2)
-		(layer "B.Cu")
-		(net "GND")
-	)
-	(segment
 		(start 102.387002 62.061)
 		(end 102.099348 62.061)
@@
 	)
 	(segment
+		(start 82.491 65.941)
+		(end 82.47 65.962)
+		(width 0.2)
+		(layer "F.Cu")
+		(net "/Speaker")
+	)
+	(segment
 		(start 99.615905 75.533062)
 		(end 98.739938 75.533062)
@@
 		(net "/Speaker")
 	)
+	(segment
+		(start 84.28 65.941)
+		(end 82.491 65.941)
+		(width 0.2)
+		(layer "F.Cu")
+		(net "/Speaker")
+	)
 	(via
 		(at 97.762 76.511)
@@
 		(net "/Speaker")
 	)
+	(via
+		(at 84.28 65.941)
+		(size 0.6)
+		(drill 0.3)
+		(layers "F.Cu" "B.Cu")
+		(net "/Speaker")
+	)
 	(segment
-		(start 87.142 65.891)
-		(end 82.47 65.891)
+		(start 84.33 65.891)
+		(end 84.28 65.941)
 		(width 0.2)
 		(layer "B.Cu")
@@
 		(width 0.2)
 		(layer "B.Cu")
+		(net "/Speaker")
+	)
+	(segment
+		(start 87.142 65.891)
+		(end 84.33 65.891)
+		(width 0.2)
+		(layer "B.Cu")

Commit message: Speaker repositioned
Parts:
- moved LS1 2.74 mm to (81.5, 60.1)
Routing:
- net /Speaker: track 22.4 -> 23.5 mm
Changed lines of the file:
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@@
 	(footprint "OWMB-404020SA-40-17:OWMB-404020SA-40-17"
 		(layer "F.Cu")
-		(at 80.47 62.596 180)
+		(at 81.486 60.056 180)
 		(property "Reference" "LS1"
 			(at -3 -4.978 180)
@@
 		(layer "User.1")
 		(pts
-			(xy 84.26222 73.561) (xy 67.262 60.861)
+			(xy 85.27822 71.021) (xy 68.278 58.321)
 		)
 		(height -22.334)
@@
 		)
 		(gr_text "12.7"
-			(at 60.77822 67.211 90)
+			(at 61.79422 64.671 90)
 			(layer "User.1")
 			(effects
@@
 	)
 	(segment
-		(start 78.47 65.962)
-		(end 78.47 64.449)
+		(start 79.486 63.422)
+		(end 79.486 61.909)
 		(width 0.2)
 		(layer "F.Cu")
@@
 	)
 	(segment
-		(start 78.47 64.449)
-		(end 78.184 64.163)
+		(start 79.486 61.909)
+		(end 79.2 61.623)
 		(width 0.2)
 		(layer "F.Cu")
@@
 	)
 	(via
-		(at 78.184 64.163)
+		(at 79.2 61.623)
 		(size 0.5842)
 		(drill 0.2032)
@@
 	)
 	(segment
-		(start 82.491 65.941)
-		(end 82.47 65.962)
+		(start 84.28 65.941)
+		(end 83.486 65.147)
 		(width 0.2)
 		(layer "F.Cu")
@@
 	)
 	(segment
-		(start 84.28 65.941)
-		(end 82.491 65.941)
+		(start 83.486 65.147)
+		(end 83.486 63.422)
 		(width 0.2)
 		(layer "F.Cu")
@@
 	)
 	(via
-		(at 97.762 76.511)
+		(at 84.28 65.941)
 		(size 0.5842)
 		(drill 0.2032)
@@
 	)
 	(via
-		(at 84.28 65.941)
-		(size 0.6)
-		(drill 0.3)
+		(at 97.762 76.511)
+		(size 0.5842)
+		(drill 0.2032)
 		(layers "F.Cu" "B.Cu")
 		(net "/Speaker")
 	)
 	(segment
-		(start 84.33 65.891)
-		(end 84.28 65.941)
+		(start 84.28 65.941)
+		(end 84.33 65.891)
 		(width 0.2)
 		(layer "B.Cu")
@@
 	)
 	(segment
-		(start 97.762 76.511)
+		(start 84.33 65.891)
 		(end 87.142 65.891)
 		(width 0.2)
@@
 	(segment
 		(start 87.142 65.891)
-		(end 84.33 65.891)
+		(end 97.762 76.511)
 		(width 0.2)
 		(layer "B.Cu")
