File: PHOBOS/PHOBOS_Control_SMA/_restore_backup_2026-10-10T22-21-48-223/PHOBOS_Control_SMA.kicad_pcb (KiCad board)
At the start: 4 copper layers, 63.4 x 78.3 mm, 90 parts, among them IC1 MPL3115A2ST1, IC10 PD2328J5050S2HF, IC4 MAPS-010144-TR0500, IC5 MAPS-010144-TR0500, IC6 MAPS-010144-TR0500, IC7 MAPS-010144-TR0500, IC8 PD2328J5050S2HF, IC9 PD2328J5050S2HF, J1 ANT3, J2 ANT4, J3 USB4056-03-A_REVA2, J4 BATT, J5 ANT1, J6 ANT2, J8 BOOT, U1 SX1280IMLTRT, U2 W25Q128JVSIQ, U3 NCP1117-3.3_SOT223, U4 RP2040, U5 TPS60403DBV, U6 LSM6DS3, Y1 C1E-52.000-10-1012-X-M, Y2 ABM8-272-T3

Commit message: SMA Version Routed (Mostly)
Parts:
- moved J1 76.8 mm to (208.1, 84.4), turned to -90 degrees
- moved J5 71.1 mm to (197.1, 111.4)
- moved J2 67.9 mm to (197.1, 84.4), turned to -90 degrees
- moved IC4 67.6 mm to (195.1, 103.4), turned to -45 degrees
- moved J6 66.9 mm to (208.1, 111.4)
- moved IC5 62.6 mm to (205.1, 103.4), turned to -45 degrees
- moved IC6 59.3 mm to (205.1, 92.4), turned to 45 degrees
- moved IC7 49.4 mm to (195.1, 92.4), turned to 45 degrees
- moved R10 45.6 mm to (190.1, 100.4), turned to 90 degrees
- moved R9 42.7 mm to (190.1, 95.9), turned to 90 degrees
- moved IC9 41.3 mm to (187.6, 100.4), turned to 90 degrees
- moved IC10 40.8 mm to (187.6, 95.9), turned to 90 degrees
- moved R2 36.5 mm to (184.6, 98.2), turned to 90 degrees
- moved IC8 33.0 mm to (182.1, 98.2), turned to 90 degrees
- moved C3 28.5 mm to (178.9, 98.2), turned to 0 degrees
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Routing:
- net -3V3: track 142.2 -> 1.98 mm, vias 6 -> 0
- net /LE4: track 66.8 -> 0.00 mm, vias 2 -> 0
- net /LE3: track 55.3 -> 0.00 mm, vias 2 -> 0
- net /SCK: track 155.3 -> 102.9 mm, vias 8 -> 5
- net /LE1: track 46.6 -> 0.00 mm, vias 2 -> 0
- net /LE2: track 43.5 -> 0.00 mm, vias 2 -> 0
- net /MOSI: track 138.5 -> 95.5 mm, vias 7 -> 5
- net GND: track 57.7 -> 22.8 mm, vias 272 -> 79
- net /P1: track 22.5 -> 3.66 mm
- net /P4: track 22.3 -> 4.49 mm
- net +3V3: track 76.0 -> 68.8 mm, vias 33 -> 25
- net /P3: track 8.01 -> 15.2 mm
- net /NSS_TRANS: track 16.1 -> 22.8 mm
- net /SCK_TRANS: track 12.8 -> 19.4 mm
- net /P2: track 7.92 -> 14.3 mm
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Other:
- board size 63.4 x 78.3 mm -> 82.3 x 35.6 mm
