File: PHOBOS/PHOBOS_Control_SMA/_restore_backup_2026-10-10T22-21-48-223/PHOBOS_Control_SMA.kicad_sch (KiCad schematic)
At the start: 90 parts, among them IC1 MPL3115A2ST1, IC10 PD2328J5050S2HF, IC4 MAPS-010144-TR0500, IC5 MAPS-010144-TR0500, IC6 MAPS-010144-TR0500, IC7 MAPS-010144-TR0500, IC8 PD2328J5050S2HF, IC9 PD2328J5050S2HF, J1 ANT3, J2 ANT4, J3 USB4056-03-A_REVA2, J4 BATT, J5 ANT1, J6 ANT2, J8 BOOT, U1 SX1280IMLTRT, U2 W25Q128JVSIQ, U3 NCP1117-3.3_SOT223, U4 RP2040, U5 TPS60403DBV, U6 LSM6DS3, Y1 C1E-52.000-10-1012-X-M, Y2 ABM8-272-T3

Commit message: SMA Version Routed (Mostly)
Other:
- moved on the sheet: C11, C12, C21, C22, C23, C24, C25, C26, C30, C31, C36, C7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
