File: PHOBOS/PHOBOS_Control_SMA/PHOBOS_Control_SMA.kicad_pcb (KiCad board)
At the start: 4 copper layers, 63.4 x 78.3 mm, 90 parts, among them IC1 MPL3115A2ST1, IC10 PD2328J5050S2HF, IC4 MAPS-010144-TR0500, IC5 MAPS-010144-TR0500, IC6 MAPS-010144-TR0500, IC7 MAPS-010144-TR0500, IC8 PD2328J5050S2HF, IC9 PD2328J5050S2HF, J1 ANT3, J2 ANT4, J3 USB4056-03-A_REVA2, J4 BATT, J5 ANT1, J6 ANT2, J8 BOOT, U1 SX1280IMLTRT, U2 W25Q128JVSIQ, U3 NCP1117-3.3_SOT223, U4 RP2040, U5 TPS60403DBV, U6 LSM6DS3, Y1 C1E-52.000-10-1012-X-M, Y2 ABM8-272-T3

Commit message: DRC errors fixed
Parts:
- removed TP1, TP2, TP3, TP4: TestPoint, Connector_Pin:Pin_D1.0mm_L10.0mm
- TP11: moved to F.Cu
- moved TP11 182.3 mm to (1.52, 1.52), turned to 0 degrees
Connections:
- IC7 pad 14: /ANT3 -> /ANT4
- J2 pad 1: /ANT3 -> /ANT4
Routing:
- net /ANT4: track 0.00 -> 8.36 mm
- net /ANT3: track 16.7 -> 8.36 mm
- net (no net): track 5.00 -> 0.00 mm
- net /P1: track 22.5 -> 24.6 mm
- net /P2: track 7.92 -> 10.0 mm
- net /P4: track 22.3 -> 24.4 mm
- net /P3: track 8.01 -> 10.1 mm
- net /SCK: track 155.3 -> 157.2 mm
- net GND: track 57.7 -> 58.9 mm
- net /LE1: track 46.6 -> 47.6 mm
- net /MOSI: track 138.5 -> 139.4 mm
