File: PHOBOS/PHOBOS_Control_SMA/PHOBOS_Control_SMA.kicad_pcb (KiCad board)
At the start: 4 copper layers, 63.4 x 78.3 mm, 87 parts, among them IC1 MPL3115A2ST1, IC10 PD2328J5050S2HF, IC4 MAPS-010144-TR0500, IC5 MAPS-010144-TR0500, IC6 MAPS-010144-TR0500, IC7 MAPS-010144-TR0500, IC8 PD2328J5050S2HF, IC9 PD2328J5050S2HF, J1 ANT3, J2 ANT4, J3 USB4056-03-A_REVA2, J4 BATT, J5 ANT1, J6 ANT2, J7 TXRX, J8 BOOT, U1 SX1280IMLTRT, U2 W25Q128JVSIQ, U3 NCP1117-3.3_SOT223, U4 RP2040, U5 TPS60403DBV, U6 LSM6DS3, Y1 C1E-52.000-10-1012-X-M, Y2 ABM8-272-T3

Commit message: Rerouted SMA traces to be more organized and not as messy
Parts:
- moved IC9 12.8 mm to (146.4, 131.4), turned to 0 degrees
- moved IC10 12.8 mm to (178.7, 131.4), turned to 0 degrees
- moved R10 11.2 mm to (146.4, 133.9), turned to 0 degrees
- moved R9 11.2 mm to (178.7, 133.9), turned to 0 degrees
Routing:
- net /RFO2: track 5.82 -> 19.2 mm
- net /RFO1: track 5.81 -> 19.1 mm
- net /P1: track 24.8 -> 12.1 mm
- net /P4: track 24.4 -> 12.0 mm
- net /P3: track 24.5 -> 12.1 mm
- net /P2: track 24.4 -> 12.0 mm
