File: PHOBOS/PHOBOS_Control_SMA/PHOBOS_Control_SMA.kicad_sch (KiCad schematic)
At the start: 90 parts, among them IC1 MPL3115A2ST1, IC10 PD2328J5050S2HF, IC4 MAPS-010144-TR0500, IC5 MAPS-010144-TR0500, IC6 MAPS-010144-TR0500, IC7 MAPS-010144-TR0500, IC8 PD2328J5050S2HF, IC9 PD2328J5050S2HF, J1 ANT3, J2 ANT4, J3 USB4056-03-A_REVA2, J4 BATT, J5 ANT1, J6 ANT2, J8 BOOT, U1 SX1280IMLTRT, U2 W25Q128JVSIQ, U3 NCP1117-3.3_SOT223, U4 RP2040, U5 TPS60403DBV, U6 LSM6DS3, Y1 C1E-52.000-10-1012-X-M, Y2 ABM8-272-T3

Commit message: DRC errors fixed
Parts:
- TP1, TP2, TP3, TP4: now left out of the parts list
Connections:
- net ANT3: no longer IC7.14 (RF_OUT), J2.1 (In)
- new net ANT4: IC7.14 (RF_OUT), J2.1 (In)

Commit message: added screw terminals for tx rx
Parts:
- added J7: TXRX, TerminalBlock_4Ucon:TerminalBlock_4Ucon_1x02_P3.50mm_Horizontal, symbol Connector:Screw_Terminal_01x02
Connections:
- net RX: now also J7.2 (Pin_2)
- net TX: now also J7.1 (Pin_1)
