File: PHOBOS/PHOBOS_Control_SMA/_restore_backup_2026-10-11T00-36-25-942/PHOBOS_Control_SMA.kicad_pcb (KiCad board)
At the start: 4 copper layers, 63.4 x 78.3 mm, 87 parts, among them IC1 MPL3115A2ST1, IC10 PD2328J5050S2HF, IC4 MAPS-010144-TR0500, IC5 MAPS-010144-TR0500, IC6 MAPS-010144-TR0500, IC7 MAPS-010144-TR0500, IC8 PD2328J5050S2HF, IC9 PD2328J5050S2HF, J1 ANT3, J2 ANT4, J3 USB4056-03-A_REVA2, J4 BATT, J5 ANT1, J6 ANT2, J7 TXRX, J8 BOOT, U1 SX1280IMLTRT, U2 W25Q128JVSIQ, U3 NCP1117-3.3_SOT223, U4 RP2040, U5 TPS60403DBV, U6 LSM6DS3, Y1 C1E-52.000-10-1012-X-M, Y2 ABM8-272-T3

Commit message: things moved around for new space
Parts:
- removed J7: TXRX, TerminalBlock_4Ucon:TerminalBlock_4Ucon_1x02_P3.50mm_Horizontal
- moved H2 11.4 mm to (184.3, 111.7)
- moved H3 10.2 mm to (134.9, 111.7)
- moved TP8 10.1 mm to (152.3, 90.6)
- moved R19 8.18 mm to (152.0, 92.4), turned to 180 degrees
- moved C37 7.84 mm to (169.8, 101.4)
- moved C38 7.84 mm to (169.8, 97.8)
- moved C39 7.84 mm to (164.4, 99.8)
- moved U5 7.84 mm to (167.3, 99.5)
- moved H4 4.78 mm to (184.3, 85.1)
- moved C12 4.18 mm to (167.1, 87.9)
- moved C26 4.18 mm to (159.4, 82.9)
- moved C11 4.17 mm to (161.9, 91.2)
- moved IC1 4.17 mm to (162.8, 87.6)
- moved U6 4.17 mm to (161.8, 83.1)
- moved TP7 4.00 mm to (157.6, 90.7)
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Routing:
- net /RX: track 23.6 -> 5.85 mm
- net /TX: track 20.2 -> 2.69 mm
- net -3V3: track 132.9 -> 142.2 mm
- net /SDA: track 18.5 -> 15.0 mm
- net /BATT_CONT: track 5.88 -> 9.05 mm
- net /SCL: track 18.3 -> 19.8 mm
- net /SCK: track 156.1 -> 157.2 mm
- net +3V3: track 76.5 -> 76.0 mm
- net GND: vias 280 -> 272
