File: DEIMOS/INSIGHT/_restore_backup_2026-10-10T23-48-26-028/INSIGHT.kicad_sch (KiCad schematic)
At the start: 78 parts, among them J1 Batt, J3 USB_C_Receptacle_USB2.0_16P, J4 Boot, J5 GND, SW3 SW_SPDT, U1 LSM6DS3, U2 MPL3115A2, U3 W25Q128JVSIQ, U4 BNO085, U5 RP2040, U6 Adafruit GPS, U7 MPM3610GQV-Z, U8 RFM95W-915S2, Y1 ABM8-272-T3, Y2 ABS07-32.768KHZ-1-T

Commit message: Updated Insight schemtic to use rfm95W
Parts:
- removed U8: RFM95W-915S2, symbol RF_Module:RFM95W-915S2
- added C32: 10u, Capacitor_SMD:C_0603_1608Metric_Pad1.08x0.95mm_HandSolder, symbol Device:C
- added C33: 22u, Capacitor_SMD:C_0603_1608Metric_Pad1.08x0.95mm_HandSolder, symbol Device:C
- added J6: Stack 1x04, Connector_PinHeader_2.54mm:PinHeader_1x08_P2.54mm_Vertical, symbol Connector_Generic:Conn_01x08
- added J7: Conn_02x05_Odd_Even, Connector_PinHeader_2.54mm:PinHeader_2x05_P2.54mm_Vertical, symbol Connector_Generic:Conn_02x05_Odd_Even
- added J8: 5V, Connector_PinHeader_1.00mm:PinHeader_1x02_P1.00mm_Vertical, symbol Connector_Generic:Conn_01x02
- added R10: 53.6k, Resistor_SMD:R_0402_1005Metric, symbol Device:R
- added R12, R9: 100k, Resistor_SMD:R_0402_1005Metric, symbol Device:R
- added R14: 19.1k, Resistor_SMD:R_0402_1005Metric, symbol Device:R
- added U11: MPM3610GQV-Z, MPM3610:QFN3p0x5p0x1p6_MPM3610_MNP, symbol 2026-05-31_23-05-25:MPM3610GQV-Z
- added U8: RFD900ux, RFD900UX, symbol RFD900ux:RFD900UX
Connections:
- net DIO0 is gone; now on net H_INTN: U5.18 (GPIO15)
- net +3V3: now also J6.1 (Pin_1)
- net +BATT: now also J7.1 (Pin_1)
- net DIO1: now also J6.6 (Pin_6); no longer U5.27 (GPIO16)
- net DIO2: now also J6.7 (Pin_7); no longer U5.28 (GPIO17)
- net GND: now also C32.2, C33.2, J6.8 (Pin_8), J7.7 (Pin_7), J8.2 (Pin_2), R10.2, R14.2, U11.12 (PGND), U11.13 (PGND), U11.14 (PGND), U11.3 (AGND), U8.14 (GND), U8.15 (GND), U8.29 (GND), U8.30 (GND)
- net MISO: now also U5.27 (GPIO16), J6.3 (Pin_3); no longer U5.15 (GPIO12)
- net MOSI: now also U5.30 (GPIO19), J6.2 (Pin_2); no longer U5.14 (GPIO11)
- net RX: now also U8.26 (SIRTX_EXT)
- net RX1: now also J7.4 (Pin_4)
- net SCL: now also J7.5 (Pin_5)
- net SDA: now also J7.3 (Pin_3)
- net TX: now also U8.25 (SIRX_EXT)
- net VB5: now also C32.1, R9.1, U11.16 (IN)
- net SCLK: now reaches U5.29 (GPIO18)
- net Mode_Sel: now reaches U5.32 (GPIO21)
- net Main_Cont: now reaches U5.38 (GPIO26_ADC0)
- net Drogue_Cont: now reaches U5.39 (GPIO27_ADC1)
- net NSS/CS renamed GPIO13
- net RESET: no longer names the net of U5.17 (GPIO14)
- net SCK renamed GPIO10
- new net: R12.2, R14.1, U11.1 (FB)
- new net: R9.2, U11.17 (EN)
- new net: R10.1, U11.18 (AAM)
- new net: U11.19 (NC), U11.20 (NC)
- new net: U11.4 (SW), U11.5 (SW), U11.6 (SW)
- new net 5V: C33.1, J8.1 (Pin_1), R12.1, U11.7 (OUT), U11.8 (OUT), U11.9 (OUT), U8.19 (+5V)
- new net NSS: U5.28 (GPIO17)
- new net RST: J6.5 (Pin_5)
- new net SCLCK: J6.4 (Pin_4)
- new net TX2: J7.2 (Pin_2)
- no-connect marks 29 -> 26
Other:
- note added: "1: This need a right angle sma port routed to it 2: Need to figure out thermal rel network 3: route a fpdi cable port for flahsing is needed 4: NC on all other pins"
- note added: "Find 3d model"
- note added: "Need to BEEF UP"
- note added: "RFD900ux"
- note added: "RFD900x Interface"
- note removed: "RFM95W"
- moved on the sheet: J1, SW3
