File: PHOBOS/PHOBOS_PAA/PHOBOS_PAA.kicad_pcb (KiCad board)
At the start: 2 copper layers, 254 x 101.6 mm, 8 parts, among them J1 ANT1, J2 ANT2, J3 ANT3, J4 ANT4

Commit message: patches centered
Parts:
- moved J1 5.07 mm to (49.3, 87.3)
- moved J2 5.07 mm to (111.8, 87.3)
- moved J3 5.07 mm to (174.3, 87.3)
- moved J4 5.07 mm to (236.8, 87.3)
